File: pcb/autochess.kicad_pcb (KiCad board)
At the start: 2 copper layers, 200 x 200 mm, 93 parts, among them J1 EDGE_LEFT, J2 EDGE_BOT, J3 Conn_02x08_Odd_Even, SW1 SW_Push, SW10 SW_Push, SW11 SW_Push, SW12 SW_Push, SW13 SW_Push, SW14 SW_Push, SW15 SW_Push, SW16 SW_Push, SW2 SW_Push, SW3 SW_Push, SW4 SW_Push, SW5 SW_Push, SW6 SW_Push, SW7 SW_Push, SW8 SW_Push, SW9 SW_Push

Commit message: PCB layout: second attempt
Parts:
- added R10: 0, Resistor_SMD:R_1206_3216Metric_Pad1.30x1.75mm_HandSolder, B.Cu at (128.0, 47.5)
- added R11: 0, Resistor_SMD:R_1206_3216Metric_Pad1.30x1.75mm_HandSolder, B.Cu at (176.2, 47.5)
- added R12: 0, Resistor_SMD:R_1206_3216Metric_Pad1.30x1.75mm_HandSolder, B.Cu at (224.2, 47.8)
- D17, D18, D19, D20, D21, D22, D23, D24, D25, D26, D27, D28, JP1, JP10, JP11, JP13, JP14, JP15, JP17, JP18, JP19, JP2, JP20, JP21, JP22, JP23, JP24, JP25, JP26, JP27, JP28, JP3, JP6, JP7, JP9: moved to B.Cu
- moved JP1 245.2 mm to (77.2, 78.5), turned to 180 degrees
- moved JP17 237.7 mm to (106.2, 45.2), turned to 90 degrees
- moved JP2 236.8 mm to (77.5, 126.5), turned to 180 degrees
- moved JP3 236.5 mm to (77.8, 174.5), turned to 180 degrees
- moved JP21 225.5 mm to (106.2, 93.5), turned to 90 degrees
- moved JP25 220.3 mm to (106.0, 141.7), turned to 90 degrees
- moved D25 209.3 mm to (109.2, 141.5), turned to 90 degrees
- moved D17 202.4 mm to (109.8, 45.0), turned to 90 degrees
- moved JP18 197.3 mm to (154.2, 44.8), turned to 90 degrees
- moved D21 197.1 mm to (109.5, 93.5), turned to 90 degrees
- moved JP6 190.5 mm to (126.2, 126.5), turned to 180 degrees
- moved JP7 187.2 mm to (126.2, 174.2), turned to 180 degrees
- moved JP22 182.0 mm to (153.8, 93.2), turned to 90 degrees
- moved JP26 172.7 mm to (153.8, 141.7), turned to 90 degrees
- moved D26 161.3 mm to (157.2, 141.5), turned to 90 degrees
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Connections:
- D18 pad 1: /COL1 -> Net-(D18-K)
- D19 pad 1: /COL1 -> Net-(D19-K)
- D20 pad 1: /COL1 -> Net-(D20-K)
- D21 pad 1: Net-(D21-K) -> /COL2
- D23 pad 1: Net-(D22-K) -> Net-(D23-K)
- J3 pad 11: /COL3 -> /COL2
- J3 pad 13: /COL2 -> /COL3
- J3 pad 15: /COL1 -> /COL4
- J3 pad 9: /COL4 -> /COL1
- JP18 pad 1: /COL1 -> Net-(D18-K)
- JP19 pad 1: /COL1 -> Net-(D19-K)
- JP20 pad 1: /COL1 -> Net-(D20-K)
- JP21 pad 1: Net-(D21-K) -> /COL2
- JP23 pad 1: Net-(D22-K) -> Net-(D23-K)
- R1 pad 1: /COL2 -> Net-(D22-K)
- R1 pad 2: Net-(D21-K) -> Net-(D23-K)
- R2 pad 1: Net-(D21-K) -> /COL2
- R3 pad 1: Net-(D22-K) -> Net-(D23-K)
Routing:
- net (no net): track 208.0 -> 0.00 mm, vias 6 -> 0
- net /COL1: track 144.1 -> 52.9 mm, vias 4 -> 0
- net Net-(D23-K): track 0.00 -> 47.3 mm
- net Net-(D27-K): track 0.00 -> 47.2 mm
- net Net-(D18-K): track 0.00 -> 47.2 mm
- net Net-(D22-K): track 0.00 -> 46.8 mm
- net Net-(D19-K): track 0.00 -> 46.5 mm
- net Net-(D26-K): track 0.00 -> 46.5 mm
- net Net-(D17-A): track 0.00 -> 46.0 mm, vias 0 -> 1
- net Net-(D18-A): track 0.00 -> 45.8 mm, vias 0 -> 1
- net Net-(D26-A): track 0.00 -> 45.6 mm, vias 0 -> 1
- net Net-(D23-A): track 0.00 -> 45.6 mm, vias 0 -> 1
- net Net-(D21-A): track 0.00 -> 45.5 mm, vias 0 -> 1
- net Net-(D28-A): track 0.00 -> 45.5 mm, vias 0 -> 1
- net Net-(D27-A): track 0.00 -> 45.5 mm, vias 0 -> 1
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