File: pcb/autochess.kicad_sch (KiCad schematic)
At the start: 92 parts, among them J1 EDGE_LEFT, J2 EDGE_BOT, J3 Conn_02x08_Odd_Even, SW1 SW_Push, SW10 SW_Push, SW11 SW_Push, SW12 SW_Push, SW13 SW_Push, SW14 SW_Push, SW15 SW_Push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

Commit message: PCB layout: second attempt
Parts:
- added R10, R11, R12: 0, Resistor_SMD:R_1206_3216Metric_Pad1.30x1.75mm_HandSolder, symbol Device:R
Connections:
- net COL1: now also J3.9 (Pin_9), R10.1; no longer D18.1 (K), D19.1 (K), D20.1 (K), J3.15 (Pin_15), JP18.1 (A), JP19.1 (A), JP20.1 (A)
- net COL2: now also D21.1 (K), J3.11 (Pin_11), JP21.1 (A), R2.1; no longer J3.13 (Pin_13), R1.1
- net COL3: now also J3.13 (Pin_13); no longer J3.11 (Pin_11)
- net COL4: now also J3.15 (Pin_15); no longer J3.9 (Pin_9)
- net at D23.1 (K), JP23.1 (A), R3.1: now also R1.2; no longer D22.1 (K), JP22.1 (A), R2.2
- new net: D22.1 (K), JP22.1 (A), R1.1, R2.2
- new net: D18.1 (K), JP18.1 (A), R10.2, R11.1
- new net: D19.1 (K), JP19.1 (A), R11.2, R12.1
- new net: D20.1 (K), JP20.1 (A), R12.2
Other:
- moved on the sheet: R1
