File: pcb/proto/autochess_proto.kicad_pcb (KiCad board)
At the start: 2 copper layers, 113 x 94 mm, 17 parts, among them U1 DRV5033AJxDBZ, U2 DRV5033AJxDBZ, U3 DRV5033AJxDBZ, U4 DRV5033AJxDBZ

Commit message: Final changes in the Proto PCB
Parts:
- added REF**: MountingHole_3.2mm_M3, MountingHole:MountingHole_3.2mm_M3, F.Cu at (138.0, 138.0)
- added REF**: MountingHole_3.2mm_M3, MountingHole:MountingHole_3.2mm_M3, F.Cu at (52.0, 52.0)
- added REF**: MountingHole_3.2mm_M3, MountingHole:MountingHole_3.2mm_M3, F.Cu at (138.0, 52.0)
- added REF**: MountingHole_3.2mm_M3, MountingHole:MountingHole_3.2mm_M3, F.Cu at (52.0, 138.0)
