File: pcb/v1/autochess_v1/autochess_v1.kicad_pcb (KiCad board)
At the start: 2 copper layers, 297 parts, among them J1 Pi_Zero, J2 POWER_IN, J3 ICSP, J4 LCD_SOCKET, J5 BUTTONS, J6 SPARE, J7 POWER_IN_EXT, J8 POWER_SW2, Q1 BS170, Q2 BS170, Q3 BS170, Q4 BS170, Q5 BS170, Q6 BS170, Q7 BS170, Q8 BS170, SW1 POWER_SW1, SW2 RPI_POWER, U1 ATmega644P-20P, U10 DRV5033A, U11 DRV5033A, U12 DRV5033A, U13 DRV5033A, U14 DRV5033A, U15 DRV5033A, U16 DRV5033A, U17 DRV5033A, U18 DRV5033A, U19 DRV5033A, U2 DRV5033A, U20 DRV5033A, U21 DRV5033A, U22 DRV5033A, U23 DRV5033A, U24 DRV5033A, U25 DRV5033A, U26 DRV5033A, U27 DRV5033A, U28 DRV5033A, U29 DRV5033A, U3 DRV5033A, U30 DRV5033A, U31 DRV5033A, U32 DRV5033A, U33 DRV5033A, U34 DRV5033A, U35 DRV5033A, U36 DRV5033A, U37 DRV5033A, U38 DRV5033A, U39 DRV5033A, U4 DRV5033A, U40 DRV5033A, U41 DRV5033A, U42 DRV5033A, U43 DRV5033A, U44 DRV5033A, U45 DRV5033A, U46 DRV5033A, U47 DRV5033A, U48 DRV5033A, U49 DRV5033A, U5 DRV5033A, U50 DRV5033A, U51 DRV5033A, U52 DRV5033A, U53 DRV5033A, U54 DRV5033A, U55 DRV5033A, U56 DRV5033A, U57 DRV5033A, U58 DRV5033A, U59 DRV5033A, U6 DRV5033A, U60 DRV5033A, U61 DRV5033A, U62 DRV5033A, U63 DRV5033A, U64 DRV5033A, U65 DRV5033A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

Commit message: Misc. PCB changes
Parts:
- moved SW1 481.9 mm to (64.0, 368.0), turned to 90 degrees
- moved J1 395.0 mm to (123.0, 362.0), turned to 90 degrees
- moved Q8 383.9 mm to (247.1, 437.9)
- moved C1 383.9 mm to (125.6, 483.5)
- moved C11 383.9 mm to (125.6, 517.0)
- moved C12 383.9 mm to (131.6, 483.5)
- moved C13 383.9 mm to (131.6, 486.9)
- moved C14 383.9 mm to (131.6, 490.2)
- moved C15 383.9 mm to (131.6, 493.6)
- moved C17 383.9 mm to (131.6, 500.2)
- moved C18 383.9 mm to (131.6, 503.6)
- moved C19 383.9 mm to (131.6, 506.9)
- moved C2 383.9 mm to (125.6, 486.9)
- moved C20 383.9 mm to (131.6, 510.3)
- moved C22 383.9 mm to (131.6, 517.0)
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
Commit message: Continue laying out the PCB
Parts:
- removed C133: 10uF, Capacitor_SMD:C_1206_3216Metric_Pad1.33x1.80mm_HandSolder
- removed C134, C135: 22pF, Capacitor_SMD:C_1206_3216Metric_Pad1.33x1.80mm_HandSolder
- removed J6: SPARE, Connector_PinHeader_2.54mm:PinHeader_1x07_P2.54mm_Vertical
- removed R10: 10K, Resistor_SMD:R_1206_3216Metric_Pad1.30x1.75mm_HandSolder
- removed R11: 1K, Resistor_SMD:R_1206_3216Metric_Pad1.30x1.75mm_HandSolder
- removed SW2: RPI_POWER, Jumper:SolderJumper-2_P1.3mm_Open_TrianglePad1.0x1.5mm
- removed the U2 at (192.0, 467.9)
- removed Y1: 20MHz, Crystal:Crystal_HC49-U_Vertical
- J1: value Pi_Zero -> CONN1; footprint Connector_PinHeader_2.54mm:PinHeader_2x20_P2.54mm_Vertical -> Connector_PinHeader_2.54mm:PinHeader_1x12_P2.54mm_Vertical
- J3: value ICSP -> CONN2; footprint Connector_IDC:IDC-Header_2x05_P2.54mm_Horizontal -> Connector_PinHeader_2.54mm:PinHeader_1x12_P2.54mm_Vertical
- J4: value LCD_SOCKET -> CONN3; footprint Connector_PinHeader_2.54mm:PinHeader_1x06_P2.54mm_Vertical -> Connector_PinHeader_2.54mm:PinHeader_1x12_P2.54mm_Vertical
- J5: value BUTTONS -> CONN4; footprint Connector_PinHeader_2.54mm:PinHeader_2x03_P2.54mm_Vertical -> Connector_PinHeader_2.54mm:PinHeader_1x12_P2.54mm_Vertical
- Q1, Q2, Q3, Q4, Q5, Q6, Q7, Q8: value BS170 -> 2N7002; footprint Package_TO_SOT_THT:TO-92_Inline -> Package_TO_SOT_SMD:SOT-23
- U1: value ATmega644P-20P -> DRV5033A; footprint Package_DIP:DIP-40_W15.24mm -> Package_TO_SOT_SMD:SOT-23
- moved D8 458.1 mm to (331.3, 68.7), turned to 180 degrees
- moved D7 436.5 mm to (293.7, 68.7), turned to 180 degrees
- moved U2 417.5 mm to (106.5, 63.8)
- moved D6 417.3 mm to (256.2, 68.7), turned to 180 degrees
- moved C1 414.7 mm to (68.7, 72.8), turned to 180 degrees
- moved D5 400.6 mm to (218.8, 68.8), turned to 180 degrees
- moved C67 390.0 mm to (68.8, 60.8)
- moved D4 387.3 mm to (181.2, 68.7), turned to 180 degrees
- moved D9 381.1 mm to (331.3, 105.7)
- moved D16 378.7 mm to (68.8, 105.7)
- moved D3 377.2 mm to (143.7, 68.7), turned to 180 degrees
- moved U1 376.4 mm to (68.8, 63.8), turned to 0 degrees
- moved D24 374.4 mm to (331.2, 143.8), turned to 180 degrees
- moved D2 370.7 mm to (106.2, 68.7), turned to 180 degrees
- moved D10 369.2 mm to (293.8, 105.7)
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- renumbered D19 to D18, D21 to D19, D23 to D20, D25 to D21, D27 to D22, D29 to D23, D31 to D24, D18 to D25, D20 to D26, D22 to D27, D24 to D28, D26 to D29, D28 to D30, D30 to D31, D35 to D33, D39 to D34, D43 to D35, D47 to D36, D51 to D37, D55 to D38, D59 to D39, D63 to D40, D36 to D41, D40 to D42, D44 to D43, D48 to D44, D52 to D45, D56 to D46, D60 to D47, D64 to D48, D33 to D49, D37 to D50, D41 to D51, D45 to D52, D49 to D53, D53 to D54, D57 to D55, D61 to D56, D34 to D57, D38 to D58, D42 to D59, D46 to D60, D50 to D61, D54 to D62, D58 to D63, D62 to D64, U11 to U10, U12 to U11, U13 to U12, U14 to U13, U15 to U14, U16 to U15, U17 to U16, U18 to U17, U20 to U18, U22 to U19, U3 to U2, U24 to U20, U26 to U21, U28 to U22, U30 to U23, U32 to U24, U19 to U25, U21 to U26, U23 to U27, U25 to U28, U27 to U29, U4 to U3, U29 to U30, U33 to U32, U34 to U33, U38 to U34, U42 to U35, U46 to U36, U50 to U37, U54 to U38, U58 to U39, U5 to U4, U62 to U40, U35 to U41, U39 to U42, U47 to U44, U51 to U45, U55 to U46, U59 to U47, U63 to U48, U36 to U49, U6 to U5, U40 to U50, U44 to U51, U48 to U52, U52 to U53, U56 to U54, U60 to U55, U64 to U56, U37 to U57, U41 to U58, U45 to U59, U7 to U6, U49 to U60, U53 to U61, U57 to U62, U61 to U63, U65 to U64, U8 to U7, U9 to U8, U10 to U9
Connections:
- J1 pad 1: unconnected-(J1-3V3-Pad1)_1 -> GND
- J1 pad 10: /MCU_TX -> /SENSOR_ON_7
- J1 pad 11: Net-(J1-GPIO17) -> /SENSOR_ON_8
- J1 pad 12: unconnected-(J1-GPIO18/PWM0-Pad12) -> GND
- J1 pad 2: Net-(SW2-A) -> +3.3V
- J1 pad 3: unconnected-(J1-SDA/GPIO2-Pad3) -> VCC
- J1 pad 4: Net-(SW2-A) -> /SENSOR_ON_1
- J1 pad 5: unconnected-(J1-SCL/GPIO3-Pad5) -> /SENSOR_ON_2
- J1 pad 6: GND -> /SENSOR_ON_3
- J1 pad 7: unconnected-(J1-GCLK0/GPIO4-Pad7) -> /SENSOR_ON_4
- J1 pad 8: /MCU_RX -> /SENSOR_ON_5
- J1 pad 9: GND -> /SENSOR_ON_6
- J3 pad 1: /MCU_MOSI -> GND
- J3 pad 10: GND -> /SENSOR_OUT_7
- J3 pad 3: unconnected-(J3-Pin_3-Pad3) -> /LED_DI
- J3 pad 4: GND -> /SENSOR_OUT_1
- J3 pad 5: /~{MCU_RESET} -> /SENSOR_OUT_2
- J3 pad 6: GND -> /SENSOR_OUT_3
- J3 pad 7: /MCU_SCK -> /SENSOR_OUT_4
- J3 pad 8: GND -> /SENSOR_OUT_5
- J3 pad 9: /MCU_MISO -> /SENSOR_OUT_6
- J4 pad 3: /LCD_SCK -> VCC
- J4 pad 4: /LCD_MISO -> /SENSOR_ON_1
- J4 pad 5: /LCD_MOSI -> /SENSOR_ON_2
- J4 pad 6: /LCD_CS -> /SENSOR_ON_3
- J5 pad 1: /BTN_1 -> GND
- J5 pad 2: GND -> +3.3V
- J5 pad 3: /BTN_2 -> /LED_DI
- J5 pad 4: GND -> /SENSOR_OUT_1
- J5 pad 5: /BTN_3 -> /SENSOR_OUT_2
- J5 pad 6: GND -> /SENSOR_OUT_3
- Q1 pad 1: Net-(Q1-D) -> /SENSOR_ON_1
- Q1 pad 2: /sensors/SENSOR_ON_1 -> GND
- Q1 pad 3: GND -> Net-(Q1-D)
- Q2 pad 1: Net-(Q2-D) -> /SENSOR_ON_2
- Q2 pad 2: /sensors/SENSOR_ON_2 -> GND
- Q2 pad 3: GND -> Net-(Q2-D)
- Q3 pad 1: Net-(Q3-D) -> /SENSOR_ON_3
- Q3 pad 2: /sensors/SENSOR_ON_3 -> GND
- Q3 pad 3: GND -> Net-(Q3-D)
- Q4 pad 1: Net-(Q4-D) -> /SENSOR_ON_4
- Q4 pad 2: /sensors/SENSOR_ON_4 -> GND
- Q4 pad 3: GND -> Net-(Q4-D)
- Q5 pad 1: Net-(Q5-D) -> /SENSOR_ON_5
- Q5 pad 2: /sensors/SENSOR_ON_5 -> GND
- Q5 pad 3: GND -> Net-(Q5-D)
- Q6 pad 1: Net-(Q6-D) -> /SENSOR_ON_6
- Q6 pad 2: /sensors/SENSOR_ON_6 -> GND
- Q6 pad 3: GND -> Net-(Q6-D)
- Q7 pad 1: Net-(Q7-D) -> /SENSOR_ON_7
- Q7 pad 2: /sensors/SENSOR_ON_7 -> GND
- Q7 pad 3: GND -> Net-(Q7-D)
- Q8 pad 1: Net-(Q8-D) -> /SENSOR_ON_8
- Q8 pad 2: /sensors/SENSOR_ON_8 -> GND
- Q8 pad 3: GND -> Net-(Q8-D)
- R1 pad 1: Net-(U1-PB0) -> /LED_DI
- R2 pad 1: /sensors/SENSOR_ON_1 -> /SENSOR_ON_1
- R3 pad 1: /sensors/SENSOR_ON_2 -> /SENSOR_ON_2
- R4 pad 1: /sensors/SENSOR_ON_3 -> /SENSOR_ON_3
- R5 pad 1: /sensors/SENSOR_ON_4 -> /SENSOR_ON_4
- R6 pad 1: /sensors/SENSOR_ON_5 -> /SENSOR_ON_5
- R7 pad 1: /sensors/SENSOR_ON_6 -> /SENSOR_ON_6
- R8 pad 1: /sensors/SENSOR_ON_7 -> /SENSOR_ON_7
- R9 pad 1: /sensors/SENSOR_ON_8 -> /SENSOR_ON_8
- U1 pad 1: Net-(U1-PB0) -> +3.3V
- U1 pad 2: /BTN_1 -> /SENSOR_OUT_1
- U1 pad 3: /BTN_2 -> Net-(Q1-D)
- U10 pad 2: /sensors/SENSOR_OUT_2 -> /SENSOR_OUT_2
- U11 pad 2: /sensors/SENSOR_OUT_3 -> /SENSOR_OUT_3
- U12 pad 2: /sensors/SENSOR_OUT_4 -> /SENSOR_OUT_4
- U13 pad 2: /sensors/SENSOR_OUT_5 -> /SENSOR_OUT_5
- U14 pad 2: /sensors/SENSOR_OUT_6 -> /SENSOR_OUT_6
- U15 pad 2: /sensors/SENSOR_OUT_7 -> /SENSOR_OUT_7
- U16 pad 2: /sensors/SENSOR_OUT_8 -> /SENSOR_OUT_8
- U17 pad 2: /sensors/SENSOR_OUT_1 -> /SENSOR_OUT_1
- U18 pad 2: /sensors/SENSOR_OUT_2 -> /SENSOR_OUT_2
- U19 pad 2: /sensors/SENSOR_OUT_3 -> /SENSOR_OUT_3
- U2 pad 2: /sensors/SENSOR_OUT_2 -> /SENSOR_OUT_2
- U20 pad 2: /sensors/SENSOR_OUT_4 -> /SENSOR_OUT_4
- U21 pad 2: /sensors/SENSOR_OUT_5 -> /SENSOR_OUT_5
- U22 pad 2: /sensors/SENSOR_OUT_6 -> /SENSOR_OUT_6
- U23 pad 2: /sensors/SENSOR_OUT_7 -> /SENSOR_OUT_7
- U24 pad 2: /sensors/SENSOR_OUT_8 -> /SENSOR_OUT_8
- U25 pad 2: /sensors/SENSOR_OUT_1 -> /SENSOR_OUT_1
- U26 pad 2: /sensors/SENSOR_OUT_2 -> /SENSOR_OUT_2
- U27 pad 2: /sensors/SENSOR_OUT_3 -> /SENSOR_OUT_3
- U28 pad 2: /sensors/SENSOR_OUT_4 -> /SENSOR_OUT_4
- U29 pad 2: /sensors/SENSOR_OUT_5 -> /SENSOR_OUT_5
- U3 pad 2: /sensors/SENSOR_OUT_3 -> /SENSOR_OUT_3
- U30 pad 2: /sensors/SENSOR_OUT_6 -> /SENSOR_OUT_6
- U31 pad 2: /sensors/SENSOR_OUT_7 -> /SENSOR_OUT_7
- U32 pad 2: /sensors/SENSOR_OUT_8 -> /SENSOR_OUT_8
- U33 pad 2: /sensors/SENSOR_OUT_1 -> /SENSOR_OUT_1
- U34 pad 2: /sensors/SENSOR_OUT_2 -> /SENSOR_OUT_2
- U35 pad 2: /sensors/SENSOR_OUT_3 -> /SENSOR_OUT_3
- U36 pad 2: /sensors/SENSOR_OUT_4 -> /SENSOR_OUT_4
- U37 pad 2: /sensors/SENSOR_OUT_5 -> /SENSOR_OUT_5
- U38 pad 2: /sensors/SENSOR_OUT_6 -> /SENSOR_OUT_6
- U39 pad 2: /sensors/SENSOR_OUT_7 -> /SENSOR_OUT_7
- U4 pad 2: /sensors/SENSOR_OUT_4 -> /SENSOR_OUT_4
- U40 pad 2: /sensors/SENSOR_OUT_8 -> /SENSOR_OUT_8
- U41 pad 2: /sensors/SENSOR_OUT_1 -> /SENSOR_OUT_1
- U42 pad 2: /sensors/SENSOR_OUT_2 -> /SENSOR_OUT_2
- U43 pad 2: /sensors/SENSOR_OUT_3 -> /SENSOR_OUT_3
- U44 pad 2: /sensors/SENSOR_OUT_4 -> /SENSOR_OUT_4
- U45 pad 2: /sensors/SENSOR_OUT_5 -> /SENSOR_OUT_5
- U46 pad 2: /sensors/SENSOR_OUT_6 -> /SENSOR_OUT_6
- U47 pad 2: /sensors/SENSOR_OUT_7 -> /SENSOR_OUT_7
- U48 pad 2: /sensors/SENSOR_OUT_8 -> /SENSOR_OUT_8
- U49 pad 2: /sensors/SENSOR_OUT_1 -> /SENSOR_OUT_1
- U5 pad 2: /sensors/SENSOR_OUT_5 -> /SENSOR_OUT_5
- U50 pad 2: /sensors/SENSOR_OUT_2 -> /SENSOR_OUT_2
- U51 pad 2: /sensors/SENSOR_OUT_3 -> /SENSOR_OUT_3
- U52 pad 2: /sensors/SENSOR_OUT_4 -> /SENSOR_OUT_4
- U53 pad 2: /sensors/SENSOR_OUT_5 -> /SENSOR_OUT_5
- U54 pad 2: /sensors/SENSOR_OUT_6 -> /SENSOR_OUT_6
- U55 pad 2: /sensors/SENSOR_OUT_7 -> /SENSOR_OUT_7
- U56 pad 2: /sensors/SENSOR_OUT_8 -> /SENSOR_OUT_8
- U57 pad 2: /sensors/SENSOR_OUT_1 -> /SENSOR_OUT_1
- U58 pad 2: /sensors/SENSOR_OUT_2 -> /SENSOR_OUT_2
- U59 pad 2: /sensors/SENSOR_OUT_3 -> /SENSOR_OUT_3
- U6 pad 2: /sensors/SENSOR_OUT_6 -> /SENSOR_OUT_6
- U60 pad 2: /sensors/SENSOR_OUT_4 -> /SENSOR_OUT_4
- U61 pad 2: /sensors/SENSOR_OUT_5 -> /SENSOR_OUT_5
- U62 pad 2: /sensors/SENSOR_OUT_6 -> /SENSOR_OUT_6
- U63 pad 2: /sensors/SENSOR_OUT_7 -> /SENSOR_OUT_7
- U64 pad 2: /sensors/SENSOR_OUT_8 -> /SENSOR_OUT_8
- U7 pad 2: /sensors/SENSOR_OUT_7 -> /SENSOR_OUT_7
- U8 pad 2: /sensors/SENSOR_OUT_8 -> /SENSOR_OUT_8
- U9 pad 2: /sensors/SENSOR_OUT_1 -> /SENSOR_OUT_1
Routing:
- added copper zone on B.Cu, net GND
- added copper zone on F.Cu, net GND

Commit message: Continue laying out the PCB
Parts:
- moved C8 480.5 mm to (331.2, 72.8), turned to 180 degrees
- moved C7 462.5 mm to (293.8, 72.8), turned to 180 degrees
- moved U8 457.1 mm to (331.3, 63.8)
- moved C6 447.0 mm to (256.2, 72.8), turned to 180 degrees
- moved U7 442.7 mm to (293.8, 63.8)
- moved C5 434.3 mm to (218.7, 72.8), turned to 180 degrees
- moved U6 431.3 mm to (256.2, 63.8)
- moved C4 424.5 mm to (181.2, 72.8), turned to 180 degrees
- moved U5 422.8 mm to (218.8, 63.8)
- moved C3 417.8 mm to (143.8, 72.8), turned to 180 degrees
- moved U4 417.7 mm to (181.2, 63.8)
- moved C74 417.0 mm to (331.2, 60.8)
- moved U3 415.9 mm to (143.8, 63.8)
- moved C2 414.6 mm to (106.2, 72.8), turned to 180 degrees
- moved C9 404.6 mm to (68.8, 109.8)
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
Commit message: Continue layout
Parts:
- moved C11 407.9 mm to (143.8, 109.5)
- moved C13 387.0 mm to (218.8, 109.8)
- moved U13 385.9 mm to (219.0, 100.5)
- moved U12 381.1 mm to (181.5, 100.5)
- moved U11 380.1 mm to (143.9, 100.5)
- moved C12 377.0 mm to (181.2, 109.8)
- moved C77 369.7 mm to (143.9, 97.5)
- moved C79 337.0 mm to (219.0, 97.5)
- moved C78 333.5 mm to (181.5, 97.5)
- moved R1 160.0 mm to (304.4, 428.0)
- moved F1 158.2 mm to (294.0, 430.5)
- moved C100 13.3 mm to (217.1, 419.0)
- moved C102 13.3 mm to (217.1, 425.7)
- moved C104 13.3 mm to (217.1, 432.4)
- moved C105 13.3 mm to (217.1, 435.8)
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
Commit message: Spreasheet-driven layout
Parts:
- moved C8 494.1 mm to (115.3, 517.1), turned to 0 degrees
- moved C7 475.7 mm to (115.3, 513.7), turned to 0 degrees
- moved C74 463.6 mm to (182.2, 499.7)
- moved C6 459.8 mm to (115.3, 510.4), turned to 0 degrees
- moved C73 449.7 mm to (182.2, 496.4)
- moved C5 446.4 mm to (115.3, 507.0), turned to 0 degrees
- moved C72 438.6 mm to (182.2, 493.0)
- moved C4 436.0 mm to (115.3, 503.7), turned to 0 degrees
- moved U8 433.5 mm to (186.6, 472.4)
- moved C67 430.7 mm to (182.2, 476.3)
- moved C71 430.5 mm to (182.2, 489.7)
- moved C3 428.5 mm to (115.3, 500.3), turned to 0 degrees
- moved C68 425.7 mm to (182.2, 479.6)
- moved C70 425.6 mm to (182.2, 486.3)
- moved C2 424.3 mm to (115.3, 497.0), turned to 0 degrees
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
Commit message: Continue placing component
Parts:
- moved C8 494.1 mm to (331.4, 72.8), turned to 180 degrees
- moved C7 475.8 mm to (293.9, 72.8), turned to 180 degrees
- moved C6 459.8 mm to (256.4, 72.8), turned to 180 degrees
- moved C16 449.0 mm to (331.4, 110.2)
- moved C5 446.5 mm to (218.9, 72.8), turned to 180 degrees
- moved C4 436.0 mm to (181.4, 72.8), turned to 180 degrees
- moved U8 433.5 mm to (331.2, 63.8)
- moved C15 429.6 mm to (293.9, 110.2)
- moved C3 428.5 mm to (143.9, 72.8), turned to 180 degrees
- moved C2 424.3 mm to (106.4, 72.8), turned to 180 degrees
- moved C1 423.4 mm to (68.9, 72.8), turned to 180 degrees
- moved U7 418.1 mm to (293.8, 63.8)
- moved C11 417.9 mm to (143.9, 110.2)
- moved C10 413.6 mm to (106.4, 110.2)
- moved C14 412.8 mm to (256.4, 110.2)
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