File: pcb/v1/autochess_v1/autochess_v1.kicad_pcb (KiCad board)
At the start: 2 copper layers, 288 parts, among them J1 CONN1, J2 POWER_IN, J3 CONN2, J4 CONN3, J5 CONN4, J7 POWER_IN_EXT, J8 POWER_SW2, Q1 2N7002, Q2 2N7002, Q3 2N7002, Q4 2N7002, Q5 2N7002, Q6 2N7002, Q7 2N7002, Q8 2N7002, SW1 POWER_SW1, U1 DRV5033A, U10 DRV5033A, U11 DRV5033A, U12 DRV5033A, U13 DRV5033A, U14 DRV5033A, U15 DRV5033A, U16 DRV5033A, U17 DRV5033A, U18 DRV5033A, U19 DRV5033A, U2 DRV5033A, U20 DRV5033A, U21 DRV5033A, U22 DRV5033A, U23 DRV5033A, U24 DRV5033A, U25 DRV5033A, U26 DRV5033A, U27 DRV5033A, U28 DRV5033A, U29 DRV5033A, U3 DRV5033A, U30 DRV5033A, U31 DRV5033A, U32 DRV5033A, U33 DRV5033A, U34 DRV5033A, U35 DRV5033A, U36 DRV5033A, U37 DRV5033A, U38 DRV5033A, U39 DRV5033A, U4 DRV5033A, U40 DRV5033A, U41 DRV5033A, U42 DRV5033A, U43 DRV5033A, U44 DRV5033A, U45 DRV5033A, U46 DRV5033A, U47 DRV5033A, U48 DRV5033A, U49 DRV5033A, U5 DRV5033A, U50 DRV5033A, U51 DRV5033A, U52 DRV5033A, U53 DRV5033A, U54 DRV5033A, U55 DRV5033A, U56 DRV5033A, U57 DRV5033A, U58 DRV5033A, U59 DRV5033A, U6 DRV5033A, U60 DRV5033A, U61 DRV5033A, U62 DRV5033A, U63 DRV5033A, U64 DRV5033A, U66 AMS1117-3.3, U7 DRV5033A, U8 DRV5033A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

Commit message: Place most components
Parts:
- removed J5: CONN4, Connector_PinHeader_2.54mm:PinHeader_1x12_P2.54mm_Vertical
- added J9: POWER_IN, Connector_BarrelJack:BarrelJack_Horizontal, F.Cu at (344.2, 370.5)
- J2: value POWER_IN -> CONN2; footprint Connector_BarrelJack:BarrelJack_Horizontal -> Connector_PinHeader_2.54mm:PinHeader_1x12_P2.54mm_Vertical
- J3: value CONN2 -> CONN3
- J4: value CONN3 -> CONN4
- moved C72 463.6 mm to (331.2, 60.8), turned to 180 degrees
- moved C71 449.7 mm to (293.8, 60.8), turned to 180 degrees
- moved C70 438.6 mm to (256.2, 60.8), turned to 180 degrees
- moved C65 430.7 mm to (68.8, 60.8), turned to 180 degrees
- moved C69 430.5 mm to (218.8, 60.8), turned to 180 degrees
- moved C66 425.7 mm to (106.2, 60.8), turned to 180 degrees
- moved C68 425.6 mm to (181.2, 60.8), turned to 180 degrees
- moved C67 424.0 mm to (143.8, 60.8), turned to 180 degrees
- moved C73 420.4 mm to (68.8, 98.2), turned to 180 degrees
- moved C80 416.7 mm to (331.2, 98.2), turned to 180 degrees
- moved C74 415.2 mm to (106.2, 98.2), turned to 180 degrees
- moved C75 413.3 mm to (143.8, 98.2), turned to 180 degrees
- moved C79 402.2 mm to (293.8, 98.2), turned to 180 degrees
- moved Q1 397.5 mm to (54.0, 68.8)
- moved C78 390.7 mm to (256.2, 98.2), turned to 180 degrees
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- renumbered C102 to C100, C103 to C101, C104 to C102, C105 to C103, C106 to C104, C107 to C105, C108 to C106, C109 to C107, C110 to C108, C111 to C109, C112 to C110, C113 to C111, C114 to C112, C115 to C113, C116 to C114, C117 to C115, C118 to C116, C119 to C117, C120 to C118, C121 to C119, C122 to C120, C123 to C121, C124 to C122, C125 to C123, C126 to C124, C127 to C125, C128 to C126, C129 to C127, C130 to C128, C65 to C133, C66 to C134, C67 to C65, C68 to C66, C69 to C67, C70 to C68, C71 to C69, C72 to C70, C73 to C71, C74 to C72, C75 to C73, C76 to C74, C77 to C75, C78 to C76, C79 to C77, C80 to C78, C81 to C79, C82 to C80, C83 to C81, C84 to C82, C85 to C83, C86 to C84, C87 to C85, C88 to C86, C89 to C87, C90 to C88, C91 to C89, C92 to C90, C93 to C91, C94 to C92, C95 to C93, C96 to C94, C97 to C95, C98 to C96, C99 to C97, C100 to C98, C101 to C99
Connections:
- C65 pad 1: +3.3V -> Net-(Q1-D)
- C65 pad 2: Net-(Q1-D) -> +3.3V
- J2 pad 1: Net-(J7-Pin_2) -> GND
- J2 pad 2: GND -> +3.3V
- J2 pad 3: (no net) -> /LED_DI
- J3 pad 10: /SENSOR_OUT_7 -> /SENSOR_ON_7
- J3 pad 11: /SENSOR_OUT_8 -> /SENSOR_ON_8
- J3 pad 3: /LED_DI -> VCC
- J3 pad 4: /SENSOR_OUT_1 -> /SENSOR_ON_1
- J3 pad 5: /SENSOR_OUT_2 -> /SENSOR_ON_2
- J3 pad 6: /SENSOR_OUT_3 -> /SENSOR_ON_3
- J3 pad 7: /SENSOR_OUT_4 -> /SENSOR_ON_4
- J3 pad 8: /SENSOR_OUT_5 -> /SENSOR_ON_5
- J3 pad 9: /SENSOR_OUT_6 -> /SENSOR_ON_6
- J4 pad 10: /SENSOR_ON_7 -> /SENSOR_OUT_7
- J4 pad 11: /SENSOR_ON_8 -> /SENSOR_OUT_8
- J4 pad 3: VCC -> /LED_DI
- J4 pad 4: /SENSOR_ON_1 -> /SENSOR_OUT_1
- J4 pad 5: /SENSOR_ON_2 -> /SENSOR_OUT_2
- J4 pad 6: /SENSOR_ON_3 -> /SENSOR_OUT_3
- J4 pad 7: /SENSOR_ON_4 -> /SENSOR_OUT_4
- J4 pad 8: /SENSOR_ON_5 -> /SENSOR_OUT_5
- J4 pad 9: /SENSOR_ON_6 -> /SENSOR_OUT_6
Other:
- board outline added: 316 x 368 mm

Commit message: Continue PCB layout
Parts:
- removed J7: POWER_IN_EXT, TerminalBlock_Altech:Altech_AK100_1x02_P5.00mm
- removed J8: POWER_SW2, TerminalBlock_Altech:Altech_AK100_1x02_P5.00mm
- moved R2 347.4 mm to (54.0, 64.2), turned to 90 degrees
- moved R3 317.1 mm to (54.0, 101.8), turned to 90 degrees
- moved R4 287.7 mm to (54.0, 139.2), turned to 90 degrees
- moved R5 259.5 mm to (54.0, 176.8), turned to 90 degrees
- moved R6 233.0 mm to (54.0, 214.2), turned to 90 degrees
- moved F1 216.7 mm to (331.0, 370.2)
- moved R7 208.6 mm to (54.0, 251.8), turned to 90 degrees
- moved U66 191.8 mm to (318.8, 381.0), turned to 90 degrees
- moved D65 191.8 mm to (319.0, 393.8)
- moved R8 187.4 mm to (54.0, 289.2), turned to 90 degrees
- moved R9 170.4 mm to (54.0, 326.8), turned to 90 degrees
- moved J9 0.50 mm to (344.8, 370.5)
