File: pcb/v1/autochess_v1.kicad_pcb (KiCad board)
At the start: 2 copper layers, 316 x 368 mm, 286 parts, among them J1 CONN1, J2 CONN2, J3 CONN3, J4 CONN4, J9 POWER_IN, Q1 2N7002, Q2 2N7002, Q3 2N7002, Q4 2N7002, Q5 2N7002, Q6 2N7002, Q7 2N7002, Q8 2N7002, SW1 POWER_SW1, U1 DRV5033A, U10 DRV5033A, U11 DRV5033A, U12 DRV5033A, U13 DRV5033A, U14 DRV5033A, U15 DRV5033A, U16 DRV5033A, U17 DRV5033A, U18 DRV5033A, U19 DRV5033A, U2 DRV5033A, U20 DRV5033A, U21 DRV5033A, U22 DRV5033A, U23 DRV5033A, U24 DRV5033A, U25 DRV5033A, U26 DRV5033A, U27 DRV5033A, U28 DRV5033A, U29 DRV5033A, U3 DRV5033A, U30 DRV5033A, U31 DRV5033A, U32 DRV5033A, U33 DRV5033A, U34 DRV5033A, U35 DRV5033A, U36 DRV5033A, U37 DRV5033A, U38 DRV5033A, U39 DRV5033A, U4 DRV5033A, U40 DRV5033A, U41 DRV5033A, U42 DRV5033A, U43 DRV5033A, U44 DRV5033A, U45 DRV5033A, U46 DRV5033A, U47 DRV5033A, U48 DRV5033A, U49 DRV5033A, U5 DRV5033A, U50 DRV5033A, U51 DRV5033A, U52 DRV5033A, U53 DRV5033A, U54 DRV5033A, U55 DRV5033A, U56 DRV5033A, U57 DRV5033A, U58 DRV5033A, U59 DRV5033A, U6 DRV5033A, U60 DRV5033A, U61 DRV5033A, U62 DRV5033A, U63 DRV5033A, U64 DRV5033A, U66 AMS1117-3.3, U7 DRV5033A, U8 DRV5033A, U9 DRV5033A

Commit message: WIP
Parts:
- added JP1: sw1_closed, Jumper:SolderJumper-2_P1.3mm_Bridged_Pad1.0x1.5mm, F.Cu at (338.9, 397.0)
- added R10: 0, Resistor_SMD:R_1206_3216Metric_Pad1.30x1.75mm_HandSolder, F.Cu at (338.8, 383.0)
- SW1: value POWER_SW1 -> SS11-BBIWJ-R30-R; footprint Autochess:Marquardt_1858_4205 -> easyeda2kicad:SW-TH_SS11-BBIWJ-R30-R
- moved J4 197.8 mm to (51.2, 400.8)
- moved J3 197.6 mm to (51.4, 358.8)
- moved J2 60.5 mm to (260.8, 398.2)
- moved J1 60.3 mm to (260.7, 360.2)
- moved SW1 7.22 mm to (343.1, 390.5), turned to 90 degrees
Connections:
- J9 pad 1: Net-(SW1-A) -> Net-(JP1-A)
- SW1 pad 1: Net-(SW1-A) -> Net-(JP1-B)
