File: pcb/v1/autochess_v1.kicad_sch (KiCad schematic)
At the start: 14 parts, among them J1 CONN1, J2 CONN2, J3 CONN3, J4 CONN4, J9 POWER_IN, SW1 POWER_SW1, U66 AMS1117-3.3

Commit message: WIP
Parts:
- removed SW1: POWER_SW1, Autochess:Marquardt_1858_4205, symbol Switch:SW_SPST
- added JP1: sw1_closed, Jumper:SolderJumper-2_P1.3mm_Bridged_Pad1.0x1.5mm, symbol Jumper:SolderJumper_2_Bridged
- added R10: 0, Resistor_SMD:R_1206_3216Metric_Pad1.30x1.75mm_HandSolder, symbol Device:R
- added SW1: SS11-BBIWJ-R30-R, easyeda2kicad:SW-TH_SS11-BBIWJ-R30-R, symbol easyeda2kicad:SS11-BBIWJ-R30-R
Connections:
- net at J9.1: now also JP1.1 (A), R10.2
- net at F1.1: now also SW1.2
- new net: JP1.2 (B), SW1.1
- new net: R10.1, SW1.3
Changed lines of the file:
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@@
 	)
 	(junction
+		(at 52.07 54.61)
+		(diameter 0)
+		(color 0 0 0 0)
+	)
+	(junction
 		(at 80.01 82.55)
 		(diameter 0)
@@
 	(wire
 		(pts
-			(xy 59.69 57.15) (xy 62.23 57.15)
-		)
-		(stroke
-			(width 0)
-			(type default)
-		)
-	)
-	(wire
-		(pts
 			(xy 191.77 72.39) (xy 191.77 74.93)
 		)
@@
 	(wire
 		(pts
+			(xy 52.07 54.61) (xy 52.07 57.15)
+		)
+		(stroke
+			(width 0)
+			(type default)
+		)
+	)
+	(wire
+		(pts
 			(xy 194.31 72.39) (xy 194.31 74.93)
 		)
@@
 	(wire
 		(pts
+			(xy 57.15 44.45) (xy 57.15 57.15)
+		)
+		(stroke
+			(width 0)
+			(type default)
+		)
+	)
+	(wire
+		(pts
 			(xy 181.61 30.48) (xy 184.15 30.48)
 		)
@@
 	(wire
 		(pts
+			(xy 57.15 57.15) (xy 62.23 57.15)
+		)
+		(stroke
+			(width 0)
+			(type default)
+		)
+	)
+	(wire
+		(pts
 			(xy 80.01 82.55) (xy 85.09 82.55)
 		)
@@
 	(wire
 		(pts
+			(xy 62.23 52.07) (xy 62.23 54.61)
+		)
+		(stroke
+			(width 0)
+			(type default)
+		)
+	)
+	(wire
+		(pts
 			(xy 105.41 81.28) (xy 105.41 82.55)
 		)
@@
 	(wire
 		(pts
+			(xy 52.07 54.61) (xy 62.23 54.61)
+		)
+		(stroke
+			(width 0)
+			(type default)
+		)
+	)
+	(wire
+		(pts
 			(xy 114.3 127) (xy 116.84 127)
 		)
@@
 	(wire
 		(pts
-			(xy 44.45 57.15) (xy 49.53 57.15)
+			(xy 44.45 57.15) (xy 52.07 57.15)
 		)
 		(stroke
@@
 	)
 	(symbol
+		(lib_id "easyeda2kicad:SS11-BBIWJ-R30-R")
+		(at 54.61 39.37 0)
+		(unit 1)
+		(body_style 1)
+		(exclude_from_sim no)
+		(in_bom yes)
+		(on_board yes)
+		(in_pos_files yes)
+		(dnp no)
+		(property "Reference" "SW1"
+			(at 56.83 33.02 0)
+			(show_name no)
+			(do_not_autoplace no)
+			(effects
+				(font
+					(size 1.27 1.27)
+				)
+			)
+		)
+		(property "Value" "SS11-BBIWJ-R30-R"
+			(at 56.83 35.56 0)
+			(show_name no)
+			(do_not_autoplace no)
+			(effects
+				(font
+					(size 1.27 1.27)
+				)
+			)
+		)
+		(property "Footprint" "easyeda2kicad:SW-TH_SS11-BBIWJ-R30-R"
+			(at 54.61 52.07 0)
+			(hide yes)
+			(show_name no)
+			(do_not_autoplace no)
+			(effects
+				(font
+					(size 1.27 1.27)
+				)
+			)
+		)
+		(property "Datasheet" "https://lcsc.com/product-detail/Others_Legion-SS11-BBIWJ-R30-R_C309071.html"
+			(at 54.61 54.61 0)
+			(hide yes)
+			(show_name no)
+			(do_not_autoplace no)
+			(effects
+				(font
+					(size 1.27 1.27)
+				)
+			)
+		)
+		(property "Description" ""
+			(at 54.61 39.37 0)
+			(hide yes)
+			(show_name no)
+			(do_not_autoplace no)
+			(effects
+				(font
+					(size 1.27 1.27)
+				)
+			)
+		)
+		(property "LCSC Part" "C309071"
+			(at 54.61 57.15 0)
+			(hide yes)
+			(show_name no)
+			(do_not_autoplace no)
+			(effects
+				(font
+					(size 1.27 1.27)
+				)
+			)
+		)
+		(pin "2"
+		)
+		(pin "1"
+		)
+		(pin "3"
+		)
+		(instances
+			(project "autochess_v1"
+				(path "/3df8ff08-9f77-4f65-9fed-81b599c9e86e"
+					(reference "SW1")
+					(unit 1)
+				)
+			)
+		)
+	)
+	(symbol
 		(lib_id "Connector_Generic:Conn_01x12")
 		(at 85.09 137.16 0)
@@
 	)
 	(symbol
-		(lib_id "Switch:SW_SPST")
-		(at 54.61 57.15 0)
+		(lib_id "Jumper:SolderJumper_2_Bridged")
+		(at 52.07 49.53 90)
+		(unit 1)
+		(body_style 1)
+		(exclude_from_sim no)
+		(in_bom no)
+		(on_board yes)
+		(in_pos_files yes)
+		(dnp no)
+		(property "Reference" "JP1"
+			(at 44.45 45.466 90)
+			(show_name no)
+			(do_not_autoplace no)
+			(effects
+				(font
+					(size 1.27 1.27)
+				)
+				(justify right)
+			)
+		)
+		(property "Value" "sw1_closed"
+			(at 39.878 48.006 90)
+			(show_name no)
+			(do_not_autoplace no)
+			(effects
+				(font
+					(size 1.27 1.27)
+				)
+				(justify right)
+			)
+		)
+		(property "Footprint" "Jumper:SolderJumper-2_P1.3mm_Bridged_Pad1.0x1.5mm"
+			(at 52.07 49.53 0)
+			(hide yes)
+			(show_name no)
+			(do_not_autoplace no)
+			(effects
+				(font
+					(size 1.27 1.27)
+				)
+			)
+		)
+		(property "Datasheet" ""
+			(at 58.42 49.53 0)
+			(hide yes)
+			(show_name no)
+			(do_not_autoplace no)
+			(effects
+				(font
+					(size 1.27 1.27)
+				)
+			)
+		)
+		(property "Description" "Solder Jumper, 2-pole, closed/bridged"
+			(at 57.15 49.53 0)
+			(hide yes)
+			(show_name no)
+			(do_not_autoplace no)
+			(effects
+				(font
+					(size 1.27 1.27)
+				)
+			)
+		)
+		(pin "2"
+		)
+		(pin "1"
+		)
+		(instances
+			(project "autochess_v1"
+				(path "/3df8ff08-9f77-4f65-9fed-81b599c9e86e"
+					(reference "JP1")
+					(unit 1)
+				)
+			)
+		)
+	)
+	(symbol
+		(lib_id "Device:R")
+		(at 62.23 48.26 0)
 		(unit 1)
 		(body_style 1)
@@
 		(dnp no)
 		(fields_autoplaced yes)
-		(property "Reference" "SW1"
-			(at 54.61 50.8 0)
+		(property "Reference" "R10"
+			(at 64.77 46.9899 0)
 			(show_name no)
 			(do_not_autoplace no)
@@
 					(size 1.27 1.27)
 				)
+				(justify left)
 			)
 		)
-		(property "Value" "POWER_SW1"
-			(at 54.61 53.34 0)
+		(property "Value" "0"
+			(at 64.77 49.5299 0)
 			(show_name no)
 			(do_not_autoplace no)
@@
 					(size 1.27 1.27)
 				)
+				(justify left)
 			)
 		)
-		(property "Footprint" "Autochess:Marquardt_1858_4205"
-			(at 54.61 57.15 0)
+		(property "Footprint" "Resistor_SMD:R_1206_3216Metric_Pad1.30x1.75mm_HandSolder"
+			(at 60.452 48.26 90)
 			(hide yes)
 			(show_name no)
@@
 		)
 		(property "Datasheet" ""
-			(at 54.61 57.15 0)
+			(at 62.23 48.26 0)
 			(hide yes)
 			(show_name no)
@@
 			)
 		)
-		(property "Description" "Single Pole Single Throw (SPST) switch"
-			(at 54.61 57.15 0)
+		(property "Description" "Resistor"
+			(at 62.23 48.26 0)
 			(hide yes)
 			(show_name no)
@@
 			(project "autochess_v1"
 				(path "/3df8ff08-9f77-4f65-9fed-81b599c9e86e"
-					(reference "SW1")
+					(reference "R10")
 					(unit 1)
 				)
@@
 		(in_pos_files yes)
 		(dnp no)
-		(fields_autoplaced yes)
 		(property "Reference" "F1"
-			(at 66.04 50.8 90)
+			(at 66.04 54.864 90)
 			(show_name no)
 			(do_not_autoplace no)
@@
 		)
 		(property "Value" "MF-LSMF600"
-			(at 66.04 53.34 90)
+			(at 65.024 59.944 90)
 			(show_name no)
 			(do_not_autoplace no)
