File: pcb/v1/ghostchess_v1.kicad_pcb (KiCad board)
At the start: 2 copper layers, 316 x 368 mm, 288 parts, among them J1 CONN1, J2 CONN2, J3 CONN3, J4 CONN4, J9 POWER_IN, Q1 2N7002, Q2 2N7002, Q3 2N7002, Q4 2N7002, Q5 2N7002, Q6 2N7002, Q7 2N7002, Q8 2N7002, SW1 SS11-BBIWJ-R30-R, U1 DRV5033A, U10 DRV5033A, U11 DRV5033A, U12 DRV5033A, U13 DRV5033A, U14 DRV5033A, U15 DRV5033A, U16 DRV5033A, U17 DRV5033A, U18 DRV5033A, U19 DRV5033A, U2 DRV5033A, U20 DRV5033A, U21 DRV5033A, U22 DRV5033A, U23 DRV5033A, U24 DRV5033A, U25 DRV5033A, U26 DRV5033A, U27 DRV5033A, U28 DRV5033A, U29 DRV5033A, U3 DRV5033A, U30 DRV5033A, U31 DRV5033A, U32 DRV5033A, U33 DRV5033A, U34 DRV5033A, U35 DRV5033A, U36 DRV5033A, U37 DRV5033A, U38 DRV5033A, U39 DRV5033A, U4 DRV5033A, U40 DRV5033A, U41 DRV5033A, U42 DRV5033A, U43 DRV5033A, U44 DRV5033A, U45 DRV5033A, U46 DRV5033A, U47 DRV5033A, U48 DRV5033A, U49 DRV5033A, U5 DRV5033A, U50 DRV5033A, U51 DRV5033A, U52 DRV5033A, U53 DRV5033A, U54 DRV5033A, U55 DRV5033A, U56 DRV5033A, U57 DRV5033A, U58 DRV5033A, U59 DRV5033A, U6 DRV5033A, U60 DRV5033A, U61 DRV5033A, U62 DRV5033A, U63 DRV5033A, U64 DRV5033A, U66 AMS1117-3.3, U7 DRV5033A, U8 DRV5033A, U9 DRV5033A

Commit message: Add daughter board symbol
Parts:
- moved C131 203.9 mm to (329.1, 372.0)
- moved C133 203.8 mm to (328.5, 382.9), turned to -90 degrees
- moved C134 200.6 mm to (325.5, 382.9), turned to -90 degrees
- moved C132 198.5 mm to (323.6, 372.0), turned to 180 degrees
- moved R1 77.8 mm to (52.5, 368.5), turned to 180 degrees
- moved JP1 27.7 mm to (339.0, 369.4), turned to -90 degrees
- moved U66 16.5 mm to (325.3, 365.9)
- moved R10 13.9 mm to (342.0, 369.4), turned to 90 degrees
- moved F1 12.9 mm to (335.0, 382.5), turned to 180 degrees
- moved D65 9.56 mm to (328.5, 394.8), turned to -90 degrees
- moved J9 8.14 mm to (346.0, 362.5)
- moved SW1 7.53 mm to (342.3, 383.0)

Commit message: Daughterboard footprints, more layout work
Parts:
- removed J1: CONN1, Connector_PinHeader_2.54mm:PinHeader_1x12_P2.54mm_Vertical
- removed J2: CONN2, Connector_PinHeader_2.54mm:PinHeader_1x12_P2.54mm_Vertical
- removed J3: CONN3, Connector_PinHeader_2.54mm:PinHeader_1x12_P2.54mm_Vertical
- removed J4: CONN4, Connector_PinHeader_2.54mm:PinHeader_1x12_P2.54mm_Vertical
- added X1: ~, ghostchess:GhostChess_Daughter_Board, F.Cu at (124.0, 379.0)
- added X2: ~, ghostchess:GhostChess_Daughter_Board, F.Cu at (276.0, 379.0)
- moved J9 6.54 mm to (346.0, 369.0)
- moved C131 4.46 mm to (329.1, 376.5)
- moved C132 4.46 mm to (323.6, 376.5)
- moved C133 4.46 mm to (328.5, 387.3)
- moved C134 4.46 mm to (325.5, 387.4)
- moved F1 4.46 mm to (335.0, 387.0)
- moved JP1 4.46 mm to (339.0, 373.8)
- moved R10 4.46 mm to (342.0, 373.9)
- moved U66 4.46 mm to (325.3, 370.3)
- moved SW1 4.00 mm to (342.3, 387.0)
- moved D65 3.91 mm to (331.5, 397.3)

Commit message: Continue PCB layout
Parts:
- moved R1 62.2 mm to (114.6, 365.8)
- moved C134 0.09 mm to (325.5, 387.3)
- turned C100 to 0 degrees
- turned C101 to 0 degrees
- turned C102 to 0 degrees
- turned C103 to 0 degrees
- turned C104 to 0 degrees
- turned C105 to 0 degrees
- turned C106 to 0 degrees
- turned C107 to 0 degrees
- turned C108 to 0 degrees
- turned C109 to 0 degrees
- turned C110 to 0 degrees
- turned C111 to 0 degrees
- turned C112 to 0 degrees
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Routing:
- net VCC: track 0.00 -> 760.8 mm
- net /LEDs/LED_DI: track 0.00 -> 365.0 mm
- net +3.3V: track 0.00 -> 292.4 mm
- net /SENSOR_OUT_1: track 0.00 -> 254.1 mm
- net /LED_DI: track 0.00 -> 229.4 mm
- net /SENSOR_ON_1: track 0.00 -> 219.8 mm
- net /SENSOR_ON_2: track 0.00 -> 210.8 mm
- net /SENSOR_OUT_2: track 0.00 -> 207.4 mm
- net /SENSOR_ON_3: track 0.00 -> 201.5 mm
- net /SENSOR_OUT_3: track 0.00 -> 199.1 mm
- net /SENSOR_ON_4: track 0.00 -> 192.1 mm
- net /SENSOR_OUT_4: track 0.00 -> 190.7 mm
- net /SENSOR_ON_5: track 0.00 -> 183.0 mm
- net /SENSOR_OUT_5: track 0.00 -> 182.4 mm
- net /SENSOR_ON_6: track 0.00 -> 174.3 mm
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
Commit message: Add logo
Routing:
- net VCC: track 760.8 -> 781.2 mm
- net /SENSOR_OUT_1: track 254.1 -> 259.8 mm

Commit message: Continue PCB layout
Parts:
- moved C100 159.1 mm to (68.8, 323.2)
- moved C104 159.1 mm to (218.8, 323.2)
- moved C121 159.1 mm to (181.2, 210.8)
- moved C125 159.1 mm to (331.2, 210.8)
- moved C103 106.1 mm to (218.8, 285.8)
- moved C108 106.1 mm to (106.2, 323.2)
- moved C112 106.1 mm to (256.2, 323.2)
- moved C113 106.1 mm to (143.8, 210.8)
- moved C117 106.1 mm to (293.8, 210.8)
- moved C122 106.1 mm to (181.2, 248.2)
- moved C126 106.1 mm to (331.2, 248.2)
- moved C99 106.1 mm to (68.8, 285.8)
- moved C102 53.0 mm to (218.8, 248.2)
- moved C105 53.0 mm to (106.2, 210.8)
- moved C107 53.0 mm to (106.2, 285.8)
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Connections:
- X1 pad 14: unconnected-(X1-NC-Pad14) -> /USER1
- X1 pad 15: unconnected-(X1-NC-Pad15) -> /USER2
- X1 pad 16: unconnected-(X1-NC-Pad16) -> /USER3
- X2 pad 14: unconnected-(X2-NC-Pad14) -> /USER1
- X2 pad 15: unconnected-(X2-NC-Pad15) -> /USER2
- X2 pad 16: unconnected-(X2-NC-Pad16) -> /USER3
Routing:
- net /LEDs/LED_DI: track 365.0 -> 0.00 mm
- net /SENSOR_ON_1: track 219.8 -> 560.4 mm
- net Net-(Q7-D): track 0.00 -> 318.2 mm
- net Net-(Q8-D): track 0.00 -> 313.4 mm
- net /SENSOR_ON_2: track 210.8 -> 518.0 mm
- net +3.3V: track 292.4 -> 578.0 mm, vias 0 -> 1
- net /SENSOR_ON_3: track 201.5 -> 475.6 mm
- net /SENSOR_OUT_1: track 259.8 -> 530.3 mm, vias 0 -> 6
- net /SENSOR_ON_4: track 192.1 -> 433.3 mm
- net /SENSOR_ON_5: track 183.0 -> 390.9 mm
- net /USER3: track 0.00 -> 178.6 mm
- net /SENSOR_ON_6: track 174.3 -> 346.2 mm
- net /USER2: track 0.00 -> 171.8 mm
- net /USER1: track 0.00 -> 154.3 mm
- net /SENSOR_ON_7: track 165.6 -> 305.8 mm
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