File: pcb/v1/ghostchess_v1.kicad_pcb (KiCad board)
At the start: 2 copper layers, 316 x 368 mm, 286 parts, among them J9 POWER_IN, Q1 2N7002, Q2 2N7002, Q3 2N7002, Q4 2N7002, Q5 2N7002, Q6 2N7002, Q7 2N7002, Q8 2N7002, SW1 SS11-BBIWJ-R30-R, U1 DRV5033A, U10 DRV5033A, U11 DRV5033A, U12 DRV5033A, U13 DRV5033A, U14 DRV5033A, U15 DRV5033A, U16 DRV5033A, U17 DRV5033A, U18 DRV5033A, U19 DRV5033A, U2 DRV5033A, U20 DRV5033A, U21 DRV5033A, U22 DRV5033A, U23 DRV5033A, U24 DRV5033A, U25 DRV5033A, U26 DRV5033A, U27 DRV5033A, U28 DRV5033A, U29 DRV5033A, U3 DRV5033A, U30 DRV5033A, U31 DRV5033A, U32 DRV5033A, U33 DRV5033A, U34 DRV5033A, U35 DRV5033A, U36 DRV5033A, U37 DRV5033A, U38 DRV5033A, U39 DRV5033A, U4 DRV5033A, U40 DRV5033A, U41 DRV5033A, U42 DRV5033A, U43 DRV5033A, U44 DRV5033A, U45 DRV5033A, U46 DRV5033A, U47 DRV5033A, U48 DRV5033A, U49 DRV5033A, U5 DRV5033A, U50 DRV5033A, U51 DRV5033A, U52 DRV5033A, U53 DRV5033A, U54 DRV5033A, U55 DRV5033A, U56 DRV5033A, U57 DRV5033A, U58 DRV5033A, U59 DRV5033A, U6 DRV5033A, U60 DRV5033A, U61 DRV5033A, U62 DRV5033A, U63 DRV5033A, U64 DRV5033A, U66 AMS1117-3.3, U7 DRV5033A, U8 DRV5033A, U9 DRV5033A

Commit message: More layout
Parts:
- added REF**: MountingHole_3.2mm_M3, MountingHole:MountingHole_3.2mm_M3, F.Cu at (353.0, 405.0)
- added REF**: MountingHole_3.2mm_M3, MountingHole:MountingHole_3.2mm_M3, F.Cu at (47.0, 405.0)
- added REF**: MountingHole_3.2mm_M3, MountingHole:MountingHole_3.2mm_M3, F.Cu at (47.0, 226.0)
- added REF**: MountingHole_3.2mm_M3, MountingHole:MountingHole_3.2mm_M3, F.Cu at (47.0, 47.0)
- added REF**: MountingHole_3.2mm_M3, MountingHole:MountingHole_3.2mm_M3, F.Cu at (353.0, 47.0)
- added REF**: MountingHole_3.2mm_M3, MountingHole:MountingHole_3.2mm_M3, F.Cu at (353.0, 226.0)
- moved R1 1.00 mm to (115.6, 365.8)
- turned C17 to 180 degrees
- turned C18 to 180 degrees
- turned C19 to 180 degrees
- turned C20 to 180 degrees
- turned C21 to 180 degrees
- turned C22 to 180 degrees
- turned C23 to 180 degrees
- turned C24 to 180 degrees
- turned C33 to 180 degrees
- turned C34 to 180 degrees
- turned C35 to 180 degrees
- turned C36 to 180 degrees
- turned C37 to 180 degrees
- turned C38 to 180 degrees
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Routing:
- net VCC: track 716.8 -> 3229.8 mm, vias 0 -> 9
- net +3.3V: track 578.0 -> 3045.8 mm, vias 1 -> 9
- net /SENSOR_OUT_5: track 212.3 -> 575.6 mm, vias 0 -> 8
- net /SENSOR_OUT_4: track 205.5 -> 563.9 mm, vias 0 -> 8
- net /SENSOR_OUT_8: track 232.5 -> 585.8 mm, vias 0 -> 8
- net /SENSOR_OUT_6: track 219.0 -> 567.8 mm, vias 0 -> 8
- net /LEDs/LED_DI: track 0.00 -> 345.9 mm, vias 0 -> 2
- net /SENSOR_OUT_3: track 198.8 -> 542.6 mm, vias 0 -> 8
- net /SENSOR_OUT_2: track 192.0 -> 535.8 mm, vias 0 -> 8
- net /SENSOR_OUT_7: track 225.7 -> 564.6 mm, vias 0 -> 8
- net Net-(Q3-D): track 0.00 -> 329.6 mm
- net Net-(Q4-D): track 0.00 -> 329.5 mm
- net Net-(Q2-D): track 0.00 -> 329.4 mm
- net Net-(Q5-D): track 0.00 -> 329.4 mm
- net Net-(Q6-D): track 0.00 -> 329.4 mm
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
Commit message: Fix DRC
Routing:
- net VCC: track 3229.8 -> 3236.1 mm
- net /USER2: track 171.8 -> 172.9 mm
- net /USER3: track 178.6 -> 179.6 mm
- net /SENSOR_OUT_1: track 720.1 -> 721.1 mm
- net /SENSOR_OUT_2: track 535.8 -> 536.9 mm
- net /SENSOR_OUT_3: track 542.6 -> 543.7 mm
- net /SENSOR_OUT_4: track 563.9 -> 564.9 mm
- net /SENSOR_OUT_5: track 575.6 -> 576.6 mm
- net /SENSOR_OUT_6: track 567.8 -> 568.9 mm
- net /SENSOR_OUT_7: track 564.6 -> 565.6 mm
- net /SENSOR_OUT_8: track 585.8 -> 586.8 mm
- net GND: vias 69 -> 70
