File: pcb/ghostchess_brains_v1/ghostchess_brains_v1.kicad_pcb (KiCad board)
At the start: 2 copper layers, 150 x 50 mm, 12 parts, among them J1 ISP, SW1 SW_Push, SW2 SW_Push, SW3 SW_Push, U1 ATmega644PA-P, Y1 11.0592MHz

Commit message: Start routing
Parts:
- added C3: 0.1uF, Capacitor_SMD:C_1206_3216Metric_Pad1.33x1.80mm_HandSolder, B.Cu at (93.8, 95.8)
- added C4: 0.1uF, Capacitor_SMD:C_1206_3216Metric_Pad1.33x1.80mm_HandSolder, B.Cu at (93.6, 75.0)
- added JP1: ISP_VCC, Jumper:SolderJumper-2_P1.3mm_Open_TrianglePad1.0x1.5mm, F.Cu at (161.5, 93.8)
- moved J1 9.31 mm to (164.8, 91.3)
- moved Y1 5.89 mm to (100.2, 73.3)
- moved C2 5.84 mm to (100.2, 67.6)
- moved C1 5.52 mm to (105.0, 67.5)
- moved U1 5.05 mm to (69.7, 77.8)
- moved R2 3.97 mm to (108.9, 59.3)
- moved SW1 2.50 mm to (142.5, 70.5)
- moved SW2 2.50 mm to (159.5, 70.5)
- moved SW3 2.50 mm to (176.5, 70.5)
Connections:
- J1 pad 2: VCC -> Net-(J1-Pin_2)
- U1 pad 22: /SENSOR_ON_1 -> /SENSOR_ON_8
- U1 pad 23: /SENSOR_ON_2 -> /SENSOR_ON_7
- U1 pad 24: /SENSOR_ON_3 -> /SENSOR_ON_6
- U1 pad 25: /SENSOR_ON_4 -> /SENSOR_ON_5
- U1 pad 26: /SENSOR_ON_5 -> /SENSOR_ON_4
- U1 pad 27: /SENSOR_ON_6 -> /SENSOR_ON_3
- U1 pad 28: /SENSOR_ON_7 -> /SENSOR_ON_2
- U1 pad 29: /SENSOR_ON_8 -> /SENSOR_ON_1
- U1 pad 33: /SENSOR_OUT_8 -> /SENSOR_OUT_1
- U1 pad 34: /SENSOR_OUT_7 -> /SENSOR_OUT_2
- U1 pad 35: /SENSOR_OUT_6 -> /SENSOR_OUT_3
- U1 pad 36: /SENSOR_OUT_5 -> /SENSOR_OUT_4
- U1 pad 37: /SENSOR_OUT_4 -> /SENSOR_OUT_5
- U1 pad 38: /SENSOR_OUT_3 -> /SENSOR_OUT_6
- U1 pad 39: /SENSOR_OUT_2 -> /SENSOR_OUT_7
- U1 pad 40: /SENSOR_OUT_1 -> /SENSOR_OUT_8
Routing:
- net /SENSOR_OUT_8: track 0.00 -> 74.9 mm
- net /SENSOR_OUT_7: track 0.00 -> 69.5 mm
- net /SENSOR_OUT_6: track 0.00 -> 64.1 mm
- net /SENSOR_ON_1: track 0.00 -> 60.5 mm
- net /SENSOR_ON_2: track 0.00 -> 60.0 mm
- net /SENSOR_ON_3: track 0.00 -> 59.3 mm
- net /SENSOR_ON_4: track 0.00 -> 58.8 mm
- net /SENSOR_OUT_5: track 0.00 -> 58.7 mm
- net /SENSOR_ON_7: track 0.00 -> 58.3 mm
- net /SENSOR_ON_5: track 0.00 -> 58.2 mm
- net /SENSOR_ON_6: track 0.00 -> 57.5 mm
- net /SENSOR_ON_8: track 0.00 -> 56.2 mm
- net /SENSOR_OUT_4: track 0.00 -> 53.3 mm
- net /SENSOR_OUT_3: track 0.00 -> 48.0 mm
- net /SENSOR_OUT_2: track 0.00 -> 43.7 mm
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
Commit message: brains v1 board
Parts:
- X2: footprint Display:WC1602A -> ghostchess:WC1602A_3Hole
- moved SW3 85.1 mm to (94.0, 91.5)
- moved SW2 84.2 mm to (78.0, 91.5)
- moved SW1 83.2 mm to (62.0, 91.5)
- moved C3 78.9 mm to (165.3, 62.4), turned to 0 degrees
- moved U1 76.4 mm to (145.0, 65.0)
- moved C4 75.9 mm to (169.0, 83.0), turned to 180 degrees
- moved R1 75.0 mm to (165.3, 59.5), turned to 0 degrees
- moved C1 72.9 mm to (176.9, 55.5)
- moved C2 72.8 mm to (172.0, 55.5)
- moved Y1 72.6 mm to (171.8, 61.0)
- moved R2 46.1 mm to (155.0, 61.0), turned to -90 degrees
- moved JP1 5.51 mm to (156.0, 94.1)
- moved X2 4.71 mm to (66.1, 53.0)
- moved J1 0.85 mm to (164.0, 91.5)
Connections:
- U1 pad 33: /SENSOR_OUT_1 -> /SENSOR_OUT_8
- U1 pad 34: /SENSOR_OUT_2 -> /SENSOR_OUT_7
- U1 pad 35: /SENSOR_OUT_3 -> /SENSOR_OUT_6
- U1 pad 36: /SENSOR_OUT_4 -> /SENSOR_OUT_5
- U1 pad 37: /SENSOR_OUT_5 -> /SENSOR_OUT_4
- U1 pad 38: /SENSOR_OUT_6 -> /SENSOR_OUT_3
- U1 pad 39: /SENSOR_OUT_7 -> /SENSOR_OUT_2
- U1 pad 40: /SENSOR_OUT_8 -> /SENSOR_OUT_1
Routing:
- net /BTN1: track 0.00 -> 162.5 mm
- net /BTN2: track 0.00 -> 141.1 mm
- net VCC: track 0.00 -> 126.5 mm
- net /OLED_SCL: track 0.00 -> 113.9 mm
- net /USER1: track 0.00 -> 110.8 mm
- net /BTN3: track 0.00 -> 107.7 mm
- net /USER2: track 0.00 -> 100.5 mm
- net /MOSI: track 0.00 -> 94.1 mm
- net /USER3: track 0.00 -> 90.2 mm
- net /MISO: track 0.00 -> 60.8 mm
- net /OLED_CS: track 0.00 -> 57.3 mm
- net /SENSOR_OUT_8: track 74.9 -> 30.8 mm
- net /SENSOR_OUT_7: track 69.5 -> 30.8 mm
- net /~{RESET}: track 0.00 -> 34.2 mm, vias 0 -> 1
- net /SENSOR_OUT_6: track 64.1 -> 30.8 mm
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- added copper zone on B.Cu, net GND
- added copper zone on F.Cu, net GND
Other:
- board size 150 x 50 mm -> 150 x 52 mm
- board text added: "Ghost Chess Brains v1 Ilya Strukov 2026"
