File: pcb/ghostchess_brains_v1/ghostchess_brains_v1.kicad_pcb (KiCad board)
At the start: 2 copper layers, 150 x 52 mm, 15 parts, among them J1 ISP, SW1 SW_Push, SW2 SW_Push, SW3 SW_Push, U1 ATmega644PA-P, Y1 11.0592MHz

Commit message: pcb: connect LED data to ATmega PB0
Connections:
- U1 pad 1: unconnected-(U1-PB0-Pad1) -> /LED_DI
Routing:
- net /LED_DI: track 0.00 -> 37.8 mm
Other:
- board text added: "Ghost Chess Brains v1.1 Ilya Strukov 2026"
- board text removed: "Ghost Chess Brains v1 Ilya Strukov 2026"
Changed lines of the file:
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@@
 			(remove_unused_layers no)
 			(roundrect_rratio 0.15625)
-			(net "unconnected-(U1-PB0-Pad1)")
+			(net "/LED_DI")
 			(pinfunction "PB0_1")
-			(pintype "bidirectional+no_connect")
+			(pintype "bidirectional")
 		)
 		(pad "2" thru_hole circle
@@
 		(layer "Edge.Cuts")
 	)
-	(gr_text "Ghost Chess Brains v1\nIlya Strukov 2026"
+	(gr_text "Ghost Chess Brains v1.1\nIlya Strukov 2026"
 		(at 169 58.4 0)
 		(layer "F.SilkS")
@@
 	)
 	(segment
+		(start 145 56.2)
+		(end 145 65)
+		(width 0.2)
+		(layer "F.Cu")
+		(net "/LED_DI")
+	)
+	(segment
+		(start 118.7 52.78)
+		(end 120.28 51.2)
+		(width 0.2)
+		(layer "F.Cu")
+		(net "/LED_DI")
+	)
+	(segment
+		(start 140 51.2)
+		(end 145 56.2)
+		(width 0.2)
+		(layer "F.Cu")
+		(net "/LED_DI")
+	)
+	(segment
+		(start 120.28 51.2)
+		(end 140 51.2)
+		(width 0.2)
+		(layer "F.Cu")
+		(net "/LED_DI")
+	)
+	(segment

Commit message: Brains v1.1
Parts:
- JP1: footprint Jumper:SolderJumper-2_P1.3mm_Open_TrianglePad1.0x1.5mm -> Connector_PinHeader_2.54mm:PinHeader_1x02_P2.54mm_Vertical
- moved JP1 13.7 mm to (168.0, 87.6), turned to 90 degrees
Routing:
- net VCC: track 126.5 -> 131.1 mm, vias 0 -> 1
- net Net-(J1-Pin_2): track 7.30 -> 11.9 mm
Changed lines of the file:
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@@
 		)
 	)
-	(footprint "Jumper:SolderJumper-2_P1.3mm_Open_TrianglePad1.0x1.5mm"
+	(footprint "Connector_PinHeader_2.54mm:PinHeader_1x02_P2.54mm_Vertical"
 		(layer "F.Cu")
-		(at 156 94.1 180)
-		(descr "SMD Solder Jumper, 1x1.5mm Triangular Pads, 0.3mm gap, open")
-		(tags "solder jumper open")
+		(at 168.025 87.6 90)
+		(descr "Through hole straight pin header, 1x02, 2.54mm pitch, single row")
+		(tags "Through hole pin header THT 1x02 2.54mm single row")
 		(property "Reference" "JP1"
-			(at 0 -1.8 0)
+			(at 0 -2.38 90)
 			(layer "F.SilkS")
 			(hide yes)
@@
 		)
 		(property "Value" "ISP_VCC"
-			(at 0.8 1.9 0)
+			(at 2.8 1.4 0)
 			(layer "F.SilkS")
 			(effects
@@
 		)
 		(property "Datasheet" ""
-			(at 0 0 180)
-			(unlocked yes)
+			(at 0 0 90)
 			(layer "F.Fab")
 			(hide yes)
@@
 				(font
 					(size 1.27 1.27)
-					(thickness 0.15)
 				)
 			)
 		)
 		(property "Description" "Jumper, 2-pole, open"
-			(at 0 0 180)
-			(unlocked yes)
+			(at 0 0 90)
 			(layer "F.Fab")
 			(hide yes)
@@
 				(font
 					(size 1.27 1.27)
+				)
+			)
+		)
+		(property "KiLib_Generator" "connector/pin_header_socket"
+			(at 0 0 90)
+			(layer "F.SilkS")
+			(hide yes)
+			(effects
+				(font
+					(size 1 1)
 					(thickness 0.15)
 				)
@@
 			)
 		)
-		(zone_connect 1)
-		(attr allow_soldermask_bridges)
+		(attr through_hole)
 		(duplicate_pad_numbers_are_jumpers no)
-		(fp_rect
-			(start -1.225 -0.75)
-			(end 1.225 0.75)
+		(fp_line
+			(start -1.38 -1.38)
+			(end 0 -1.38)
 			(stroke
-				(width 0)
-				(type default)
+				(width 0.12)
+				(type solid)
 			)
-			(fill yes)
-			(layer "F.Mask")
+			(layer "F.SilkS")
 		)
 		(fp_line
-			(start 1.4 1)
-			(end -1.4 1)
+			(start -1.38 0)
+			(end -1.38 -1.38)
 			(stroke
 				(width 0.12)
@@
 		)
 		(fp_line
-			(start 1.4 -1)
-			(end 1.4 1)
+			(start 1.38 1.27)
+			(end 1.38 3.92)
 			(stroke
 				(width 0.12)
@@
 		)
 		(fp_line
-			(start -1.4 1)
-			(end -1.4 -1)
+			(start -1.38 1.27)
+			(end 1.38 1.27)
 			(stroke
 				(width 0.12)
@@
 		)
 		(fp_line
-			(start -1.4 -1)
-			(end 1.4 -1)
+			(start -1.38 1.27)
+			(end -1.38 3.92)
 			(stroke
 				(width 0.12)
@@
 		)
 		(fp_line
-			(start 1.65 1.25)
-			(end 1.65 -1.25)
+			(start -1.38 3.92)
+			(end 1.38 3.92)
+			(stroke
+				(width 0.12)
+				(type solid)
+			)
+			(layer "F.SilkS")
+		)
+		(fp_rect
+			(start -1.77 -1.77)
+			(end 1.77 4.32)
 			(stroke
 				(width 0.05)
 				(type solid)
 			)
+			(fill no)
 			(layer "F.CrtYd")
 		)
 		(fp_line
-			(start 1.65 1.25)
-			(end -1.65 1.25)
+			(start 1.27 -1.27)
+			(end 1.27 3.81)
 			(stroke
-				(width 0.05)
+				(width 0.1)
 				(type solid)
 			)
-			(layer "F.CrtYd")
+			(layer "F.Fab")
 		)
 		(fp_line
-			(start -1.65 -1.25)
-			(end 1.65 -1.25)
+			(start -0.635 -1.27)
+			(end 1.27 -1.27)
 			(stroke
-				(width 0.05)
+				(width 0.1)
 				(type solid)
 			)
-			(layer "F.CrtYd")
+			(layer "F.Fab")
 		)
 		(fp_line
-			(start -1.65 -1.25)
-			(end -1.65 1.25)
+			(start -1.27 -0.635)
+			(end -0.635 -1.27)
 			(stroke
-				(width 0.05)
+				(width 0.1)
 				(type solid)
 			)
-			(layer "F.CrtYd")
+			(layer "F.Fab")
+		)
+		(fp_line
+			(start 1.27 3.81)
+			(end -1.27 3.81)
+			(stroke
+				(width 0.1)
+				(type solid)
+			)
+			(layer "F.Fab")
 		)
-		(pad "1" smd custom
-			(at -0.725 0 180)
-			(size 0.3 0.3)
-			(layers "F.Cu" "F.Mask")
+		(fp_line
+			(start -1.27 3.81)
+			(end -1.27 -0.635)
+			(stroke
+				(width 0.1)
+				(type solid)
+			)
+			(layer "F.Fab")
+		)
+		(fp_text user "${REFERENCE}"
+			(at 0 1.27 0)
+			(layer "F.Fab")
+			(effects
+				(font
+					(size 1 1)
+					(thickness 0.15)
+				)
+			)
+		)
+		(pad "1" thru_hole rect
+			(at 0 0 90)
+			(size 1.7 1.7)
+			(drill 1)
+			(layers "*.Cu" "*.Mask")
+			(remove_unused_layers no)
 			(net "Net-(J1-Pin_2)")
 			(pinfunction "A_1")
 			(pintype "passive")
-			(zone_connect 2)
-			(thermal_bridge_angle 45)
-			(options
-				(clearance outline)
-				(anchor rect)
-			)
-			(primitives
-				(gr_poly
-					(pts
-						(xy 1 0) (xy 0.5 0.75) (xy -0.5 0.75) (xy -0.5 -0.75) (xy 0.5 -0.75)
-					)
-					(width 0)
-					(fill yes)
-				)
-			)
 		)
-		(pad "2" smd custom
-			(at 0.725 0 180)
-			(size 0.3 0.3)
-			(layers "F.Cu" "F.Mask")
+		(pad "2" thru_hole circle
+			(at 0 2.54 90)
+			(size 1.7 1.7)
+			(drill 1)
+			(layers "*.Cu" "*.Mask")
+			(remove_unused_layers no)
 			(net "VCC")
 			(pinfunction "B_2")
 			(pintype "passive")
-			(zone_connect 2)
-			(thermal_bridge_angle 45)
-			(options
-				(clearance outline)
-				(anchor rect)
-			)
-			(primitives
-				(gr_poly
-					(pts
-						(xy 0.5 0.75) (xy -0.65 0.75) (xy -0.15 0) (xy -0.65 -0.75) (xy 0.5 -0.75)
-					)
-					(width 0)
-					(fill yes)
-				)
-			)
 		)
 		(embedded_fonts no)
+		(model "${KICAD10_3DMODEL_DIR}/Connector_PinHeader_2.54mm.3dshapes/PinHeader_1x02_P2.54mm_Vertical.step"
+			(offset
+				(xyz 0 0 0)
+			)
+			(scale
+				(xyz 1 1 1)
+			)
+			(rotate
+				(xyz 0 0 0)
+			)
+		)
 	)
 	(footprint "Button_Switch_THT:SW_PUSH-12mm"
@@
 			(at -5.82 -3.81 0)
 			(layer "F.SilkS")
+			(hide yes)
 			(effects
 				(font
@@
 	)
 	(segment
-		(start 156.725 94.1)
-		(end 163.94 94.1)
+		(start 164 94.04)
+		(end 163.74 94.04)
+		(width 0.5)
+		(layer "F.Cu")
+		(net "Net-(J1-Pin_2)")
+	)
+	(segment
+		(start 163.74 94.04)
+		(end 161.9 92.2)
 		(width 0.5)
 		(layer "F.Cu")
@@
 	)
 	(segment
-		(start 163.94 94.1)
-		(end 164 94.04)
+		(start 164.8 87.6)
+		(end 168.025 87.6)
+		(width 0.5)
+		(layer "F.Cu")
+		(net "Net-(J1-Pin_2)")
+	)
+	(segment
+		(start 161.9 92.2)
+		(end 161.9 90.5)
+		(width 0.5)
+		(layer "F.Cu")
+		(net "Net-(J1-Pin_2)")
+	)
+	(segment
+		(start 161.9 90.5)
+		(end 164.8 87.6)
 		(width 0.5)
 		(layer "F.Cu")
@@
 		(net "VCC")
 	)
+	(via
+		(at 170.5 84.7)
+		(size 0.6)
+		(drill 0.3)
+		(layers "F.Cu" "B.Cu")
+		(net "VCC")
+	)
 	(segment
 		(start 170.5625 67.7025)
@@
 	)
 	(segment
+		(start 170.565 83.0025)
+		(end 170.5625 83)
+		(width 0.5)
+		(layer "B.Cu")
+		(net "VCC")
+	)
+	(segment
 		(start 122.8175 59.4375)
 		(end 155 59.4375)
@@
 		(width 0.5)
 		(layer "B.Cu")
+		(net "VCC")
+	)
+	(segment
+		(start 170.565 87.6)
+		(end 170.565 83.0025)
+		(width 0.5)
+		(layer "B.Cu")
