File: pcb/ghostchess_brains_v1/ghostchess_brains_v1.kicad_sch (KiCad schematic)
At the start: 9 parts, among them J1 ISP, U1 ATmega644PA-P, Y1 10MHz

Commit message: Make progress on the brains PCB
Parts:
- removed DS1: WC1602A, Display:WC1602A, symbol Display_Character:WC1602A
- removed RV1: Contrast, symbol Device:R_Potentiometer
- added C3: 0.1uF, Capacitor_SMD:C_1206_3216Metric_Pad1.33x1.80mm_HandSolder, symbol Device:C
- added R2: 10K, Capacitor_SMD:C_1206_3216Metric_Pad1.33x1.80mm_HandSolder, symbol Device:R
- added SW1, SW2, SW3: SW_Push, Button_Switch_THT:SW_PUSH-12mm, symbol Switch:SW_Push
- added X2: (no value), Display:WC1602A, symbol ghostchess:ws0010_oled_1610
- C1, C2, R1: footprint (none) -> Capacitor_SMD:C_1206_3216Metric_Pad1.33x1.80mm_HandSolder
- J1: footprint (none) -> Connector_IDC:IDC-Header_2x05_P2.54mm_Horizontal
- X1: footprint (none) -> ghostchess:GhostChess_Daughter_Board
- Y1: value 10MHz -> 11.0592MHz; footprint (none) -> Crystal:Crystal_HC49-U_Vertical
Connections:
- net GND: now also C3.2, SW1.1, SW2.1, SW3.1, X2.1 (GND)
- net MOSI: now also X2.14 (SDI)
- net SENSOR_OUT_1: now also U1.40 (PA0); no longer U1.14 (PD0)
- net SENSOR_OUT_2: now also U1.39 (PA1); no longer U1.15 (PD1)
- net SENSOR_OUT_3: now also U1.38 (PA2); no longer U1.16 (PD2)
- net SENSOR_OUT_4: now also U1.37 (PA3); no longer U1.17 (PD3)
- net SENSOR_OUT_5: now also U1.36 (PA4); no longer U1.18 (PD4)
- net SENSOR_OUT_6: now also U1.35 (PA5); no longer U1.19 (PD5)
- net SENSOR_OUT_7: now also U1.34 (PA6); no longer U1.20 (PD6)
- net SENSOR_OUT_8: now also U1.33 (PA7); no longer U1.21 (PD7)
- net USER1: now also U1.16 (PD2)
- net USER2: now also U1.17 (PD3)
- net USER3: now also U1.18 (PD4)
- net VCC: now also C3.1, R2.1, X2.2 (VCC)
- net OLED_CS: now reaches U1.5 (PB4)
- net OLED_CS: now also R2.2, X2.16 (~{CS})
- net SCK renamed OLED_SCL
- net OLED_SCL: now also X2.12 (SCL)
- new net BTN1: SW1.2, U1.19 (PD5)
- new net BTN2: SW2.2, U1.20 (PD6)
- new net BTN3: SW3.2, U1.21 (PD7)
- new net MCU_RX: U1.14 (PD0)
- new net MCU_TX: U1.15 (PD1)
- no-connect marks 2 -> 7
Other:
- note added: "OLED: Winstar WS0010 Clone, SPI"
- note added: "TODO * Serial header * Correct MCU fuse config!"
- note removed: "TODO: 1602 LED: is it 3.3V or 5V?"
- moved on the sheet: C1, C2, J1, R1, U1, Y1

Commit message: Start routing
Parts:
- added C4: 0.1uF, Capacitor_SMD:C_1206_3216Metric_Pad1.33x1.80mm_HandSolder, symbol Device:C
- added JP1: ISP_VCC, Jumper:SolderJumper-2_P1.3mm_Open_TrianglePad1.0x1.5mm, symbol Jumper:Jumper_2_Open
Connections:
- net GND: now also C4.2
- net SENSOR_ON_1: now also U1.29 (PC7); no longer U1.22 (PC0)
- net SENSOR_ON_2: now also U1.28 (PC6); no longer U1.23 (PC1)
- net SENSOR_ON_3: now also U1.27 (PC5); no longer U1.24 (PC2)
- net SENSOR_ON_4: now also U1.26 (PC4); no longer U1.25 (PC3)
- net SENSOR_ON_5: now also U1.25 (PC3); no longer U1.26 (PC4)
- net SENSOR_ON_6: now also U1.24 (PC2); no longer U1.27 (PC5)
- net SENSOR_ON_7: now also U1.23 (PC1); no longer U1.28 (PC6)
- net SENSOR_ON_8: now also U1.22 (PC0); no longer U1.29 (PC7)
- net SENSOR_OUT_1: now also U1.33 (PA7); no longer U1.40 (PA0)
- net SENSOR_OUT_2: now also U1.34 (PA6); no longer U1.39 (PA1)
- net SENSOR_OUT_3: now also U1.35 (PA5); no longer U1.38 (PA2)
- net SENSOR_OUT_4: now also U1.36 (PA4); no longer U1.37 (PA3)
- net SENSOR_OUT_5: now also U1.37 (PA3); no longer U1.36 (PA4)
- net SENSOR_OUT_6: now also U1.38 (PA2); no longer U1.35 (PA5)
- net SENSOR_OUT_7: now also U1.39 (PA1); no longer U1.34 (PA6)
- net SENSOR_OUT_8: now also U1.40 (PA0); no longer U1.33 (PA7)
- net VCC: now also C4.1, JP1.2 (B); no longer J1.2 (Pin_2)
- new net: J1.2 (Pin_2), JP1.1 (A)

Commit message: brains v1 board
Parts:
- X2: footprint Display:WC1602A -> ghostchess:WC1602A_3Hole
Connections:
- net SENSOR_OUT_1: now also U1.40 (PA0); no longer U1.33 (PA7)
- net SENSOR_OUT_2: now also U1.39 (PA1); no longer U1.34 (PA6)
- net SENSOR_OUT_3: now also U1.38 (PA2); no longer U1.35 (PA5)
- net SENSOR_OUT_4: now also U1.37 (PA3); no longer U1.36 (PA4)
- net SENSOR_OUT_5: now also U1.36 (PA4); no longer U1.37 (PA3)
- net SENSOR_OUT_6: now also U1.35 (PA5); no longer U1.38 (PA2)
- net SENSOR_OUT_7: now also U1.34 (PA6); no longer U1.39 (PA1)
- net SENSOR_OUT_8: now also U1.33 (PA7); no longer U1.40 (PA0)
Other:
- note added: "TODO * UART header * Correct MCU fuse config!"
- note removed: "TODO * Serial header * Correct MCU fuse config!"
Changed lines of the file:
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@@
 		)
 	)
-	(text "TODO\n * Serial header\n * Correct MCU fuse config!"
+	(text "TODO\n * UART header\n * Correct MCU fuse config!"
 		(exclude_from_sim no)
 		(at 238.506 22.86 0)
@@
 	)
 	(label "SENSOR_OUT_6"
-		(at 177.8 48.26 0)
+		(at 177.8 55.88 0)
 		(effects
 			(font
@@
 	)
 	(label "SENSOR_OUT_7"
-		(at 177.8 45.72 0)
+		(at 177.8 58.42 0)
 		(effects
 			(font
@@
 	)
 	(label "SENSOR_OUT_1"
-		(at 177.8 60.96 0)
+		(at 177.8 43.18 0)
 		(effects
 			(font
@@
 	)
 	(label "SENSOR_OUT_4"
-		(at 177.8 53.34 0)
+		(at 177.8 50.8 0)
 		(effects
 			(font
@@
 	)
 	(label "SENSOR_OUT_8"
-		(at 177.8 43.18 0)
+		(at 177.8 60.96 0)
 		(effects
 			(font
@@
 	)
 	(label "SENSOR_OUT_3"
-		(at 177.8 55.88 0)
+		(at 177.8 48.26 0)
 		(effects
 			(font
@@
 	)
 	(label "SENSOR_OUT_2"
-		(at 177.8 58.42 0)
+		(at 177.8 45.72 0)
 		(effects
 			(font
@@
 	)
 	(label "SENSOR_OUT_5"
-		(at 177.8 50.8 0)
+		(at 177.8 53.34 0)
 		(effects
 			(font
@@
 			)
 		)
-		(property "Footprint" "Display:WC1602A"
+		(property "Footprint" "ghostchess:WC1602A_3Hole"
 			(at 251.46 57.15 0)
 			(hide yes)
