File: pcb/ghostchess_brains_v1/ghostchess_brains_v1.kicad_sch (KiCad schematic)
At the start: 15 parts, among them J1 ISP, SW1 SW_Push, SW2 SW_Push, SW3 SW_Push, U1 ATmega644PA-P, Y1 11.0592MHz

Commit message: pcb: connect LED data to ATmega PB0
Connections:
- net LED_DI: now also U1.1 (PB0)
- no-connect marks 7 -> 6
Changed lines of the file:
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@@
 	)
 	(no_connect
-		(at 177.8 66.04)
-	)
-	(no_connect
 		(at 147.32 58.42)
 	)
@@
 		)
 	)
+	(label "LED_DI"
+		(at 177.8 66.04 0)
+		(effects
+			(font
+				(size 1.27 1.27)
+			)
+			(justify left bottom)
+		)
+	)

Commit message: Brains v1.1
Parts:
- JP1: footprint Jumper:SolderJumper-2_P1.3mm_Open_TrianglePad1.0x1.5mm -> Connector_PinHeader_2.54mm:PinHeader_1x02_P2.54mm_Vertical
Changed lines of the file:
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@@
 			)
 		)
-		(property "Footprint" "Jumper:SolderJumper-2_P1.3mm_Open_TrianglePad1.0x1.5mm"
+		(property "Footprint" "Connector_PinHeader_2.54mm:PinHeader_1x02_P2.54mm_Vertical"
 			(at 82.55 119.38 0)
 			(hide yes)
